File: hardware/analog.kicad_sch (KiCad schematic)
At the start: 19 parts, among them J5 Conn_01x03, Q1 STT6N3LLH6, Q2 IKW40N120H3FKSA1, U6 MCP1407-E/SN, U7 SCS-200LD

Commit message: Added kicad-jlcpcb-tools compatible lcsc parts (tentative)
Parts:
- C18, C19, C20, C21: LCSC (none) -> C20613286
- D1, D2, D3, D4, D6, D9: LCSC (none) -> C3013866
- Q1: LCSC (none) -> C457495
- Q2: LCSC (none) -> C3199294
- R11, R2: LCSC (none) -> C101257
- R3: LCSC (none) -> C2792070
- R9: LCSC (none) -> C137704
- U6: LCSC (none) -> C52138
