File: hardware/analog.kicad_sch (KiCad schematic)
At the start: 19 parts, among them J5 Conn_01x03, Q1 STT6N3LLH6, Q2 IKW40N120H3FKSA1, U6 MCP1407-E/SN, U7 SCS-200LD

Commit message: Updated sheet numbers + annotatios to embed in other project
Parts:
- renumbered C18 to C1001, C19 to C1002, C20 to C1003, C21 to C1004, D1 to D1001, D2 to D1002, D3 to D1003, D4 to D1004, D6 to D1005, D9 to D1006, J5 to J1001, Q1 to Q1001, Q2 to Q1002, R11 to R1001, R2 to R1002, R3 to R1003, R9 to R1004, U7 to U1001, U6 to U1002
