File: hardware/cbank.kicad_sch (KiCad schematic)
At the start: 20 parts

Commit message: Added kicad-jlcpcb-tools compatible lcsc parts (tentative)
Parts:
- C22, C23, C24, C25, C26, C27, C28, C29, C30, C31, C32, C33, C34, C35, C36, C37, C38, C39, C40, C41: LCSC (none) -> C1021531
