File: hardware/cbank.kicad_sch (KiCad schematic)
At the start: 20 parts

Commit message: Updated sheet numbers + annotatios to embed in other project
Parts:
- renumbered C22 to C5001, C23 to C5002, C24 to C5003, C25 to C5004, C26 to C5005, C27 to C5006, C28 to C5007, C29 to C5008, C30 to C5009, C31 to C5010, C32 to C5011, C33 to C5012, C34 to C5013, C35 to C5014, C36 to C5015, C37 to C5016, C38 to C5017, C39 to C5018, C40 to C5019, C41 to C5020
