File: hardware/emfi.kicad_sch (KiCad schematic)
At the start: 10 parts, among them J1 USB_B_Micro, J2 Conn_Coaxial, J3 Conn_Coaxial, J6 Conn_Coaxial, U8 74LVC1G32

Commit message: Added kicad-jlcpcb-tools compatible lcsc parts (tentative)
Parts:
- C1, C42: LCSC (none) -> C36911393
- J1: LCSC (none) -> C2894326; Manufacturer Wurth Electronik -> Wurth Elektronik; Price 1.70 -> (none); Vendor Farnell -> (none); VendorRef 2470822 -> (none)
- J2, J3, J6: LCSC (none) -> C3175374
- L1: LCSC (none) -> C85834
- R7: LCSC (none) -> C2792070
- U8: LCSC (none) -> C12516
