File: hardware/emfi.kicad_sch (KiCad schematic)
At the start: 10 parts, among them J1 USB_B_Micro, J2 Conn_Coaxial, J3 Conn_Coaxial, J6 Conn_Coaxial, U8 74LVC1G32

Commit message: Updated sheet numbers + annotatios to embed in other project
Parts:
- renumbered C1 to C3001, C42 to C3002, J1 to J3001, J2 to J3002, J3 to J3003, J6 to J3004, L1 to L3001, LOGO1 to LOGO3001, R7 to R3001, U8 to U3001
