File: hardware/ft232.kicad_sch (KiCad schematic)
At the start: 2 parts, among them U2 FT232RL

Commit message: Added kicad-jlcpcb-tools compatible lcsc parts (tentative)
Parts:
- C9: LCSC (none) -> C36911393
- U2: LCSC (none) -> C8690
