File: hardware/ft232.kicad_sch (KiCad schematic)
At the start: 2 parts, among them U2 FT232RL

Commit message: Updated sheet numbers + annotatios to embed in other project
Parts:
- renumbered C9 to C6001, U2 to U6001
