File: hardware/mcu.kicad_sch (KiCad schematic)
At the start: 16 parts, among them J4 Conn_01x02, U1 STM32F205RETx

Commit message: Added kicad-jlcpcb-tools compatible lcsc parts (tentative)
Parts:
- C17, C2, C3, C4, C5, C6, C7, C8: LCSC (none) -> C36911393
- D7: LCSC (none) -> C598355
- D8: LCSC (none) -> C5875725
- R1, R4: LCSC (none) -> C2792070
- R10, R8: LCSC (none) -> C228008
- U1: LCSC (none) -> C66278
