File: hardware/mcu.kicad_sch (KiCad schematic)
At the start: 16 parts, among them J4 Conn_01x02, U1 STM32F205RETx

Commit message: Updated sheet numbers + annotatios to embed in other project
Parts:
- renumbered C6 to C2001, C7 to C2002, C8 to C2003, C2 to C2004, C3 to C2005, C4 to C2006, C5 to C2007, C17 to C2008, D7 to D2001, D8 to D2002, J4 to J2001, R4 to R2001, R8 to R2002, R10 to R2003, R1 to R2004, U1 to U2001
