File: hardware/power.kicad_sch (KiCad schematic)
At the start: 14 parts, among them U3 MIC2288, U4 LD1117S33TR_SOT223, U5 LD1117S33TR_SOT223

Commit message: Added kicad-jlcpcb-tools compatible lcsc parts (tentative)
Parts:
- C10, C11, C12, C13, C14, C16: LCSC (none) -> C36911393
- C15: LCSC (none) -> C6119899
- D5: LCSC (none) -> C145540
- L2: LCSC (none) -> C98022
- R5: LCSC (none) -> C137768
- R6: LCSC (none) -> C103390
- U3: LCSC (none) -> C220754
- U4, U5: LCSC (none) -> C86781
