File: hardware/power.kicad_sch (KiCad schematic)
At the start: 14 parts, among them U3 MIC2288, U4 LD1117S33TR_SOT223, U5 LD1117S33TR_SOT223

Commit message: Updated sheet numbers + annotatios to embed in other project
Parts:
- renumbered C10 to C4001, C11 to C4002, C12 to C4003, C13 to C4004, C14 to C4005, C15 to C4006, C16 to C4007, D5 to D4001, L2 to L4001, R5 to R4001, R6 to R4002, U3 to U4001, U4 to U4002, U5 to U4003
