File: hardware/emfi.kicad_pcb (KiCad board)
At the start: 2 copper layers, 132.5 x 38 mm, 81 parts, among them J1 USB_B_Micro, J2 Conn_Coaxial, J3 Conn_Coaxial, J4 Conn_01x02, J5 Conn_01x03, J6 Conn_Coaxial, Q1 STT6N3LLH6, Q2 IKW40N120H3FKSA1, U1 STM32F205RETx, U2 FT232RL, U3 MIC2288, U4 LD1117S33TR_SOT223, U5 LD1117S33TR_SOT223, U6 MCP1407-E/SN, U7 SCS-200LD, U8 74LVC1G32

Commit message: Updated sheet numbers + annotatios to embed in other project
Parts:
- renumbered C18 to C1001, C19 to C1002, C20 to C1003, C21 to C1004, C6 to C2001, C7 to C2002, C8 to C2003, C2 to C2004, C3 to C2005, C4 to C2006, C5 to C2007, C17 to C2008, C1 to C3001, C42 to C3002, C10 to C4001, C11 to C4002, C12 to C4003, C13 to C4004, C14 to C4005, C15 to C4006, C16 to C4007, C22 to C5001, C23 to C5002, C24 to C5003, C25 to C5004, C26 to C5005, C27 to C5006, C28 to C5007, C29 to C5008, C30 to C5009, C31 to C5010, C32 to C5011, C33 to C5012, C34 to C5013, C35 to C5014, C36 to C5015, C37 to C5016, C38 to C5017, C39 to C5018, C40 to C5019, C41 to C5020, C9 to C6001, D1 to D1001, D2 to D1002, D3 to D1003, D4 to D1004, D6 to D1005, D9 to D1006, D7 to D2001, D8 to D2002, D5 to D4001, J5 to J1001, J4 to J2001, J1 to J3001, J2 to J3002, J3 to J3003, J6 to J3004, L1 to L3001, L2 to L4001, LOGO1 to LOGO3001, Q1 to Q1001, Q2 to Q1002, R11 to R1001, R2 to R1002, R3 to R1003, R9 to R1004, R4 to R2001, R8 to R2002, R10 to R2003, R1 to R2004, R7 to R3001, R5 to R4001, R6 to R4002, U7 to U1001, U6 to U1002, U1 to U2001, U8 to U3001, U3 to U4001, U4 to U4002, U5 to U4003, U2 to U6001
Connections:
- net /analog/CHARGE_PWM renamed /mcu/TIM1_CH1
- net /mcu/ADC renamed /mcu/ADC123_IN0
- net /mcu/RX renamed /ft232/TX
- J3001 pad 4: Net-(J1-Pad4) -> unconnected-(J3001-ID-Pad4)
- U1002 pad 3: Net-(U6-Pad3) -> unconnected-(U1002-NC-Pad3)
- U2001 pad 10: Net-(U1-Pad10) -> unconnected-(U2001-PC2-Pad10)
- U2001 pad 11: Net-(U1-Pad11) -> unconnected-(U2001-PC3-Pad11)
- U2001 pad 15: Net-(U1-Pad15) -> unconnected-(U2001-PA1-Pad15)
- U2001 pad 16: Net-(U1-Pad16) -> unconnected-(U2001-PA2-Pad16)
- U2001 pad 17: Net-(U1-Pad17) -> unconnected-(U2001-PA3-Pad17)
- U2001 pad 20: Net-(U1-Pad20) -> unconnected-(U2001-PA4-Pad20)
- U2001 pad 21: Net-(U1-Pad21) -> unconnected-(U2001-PA5-Pad21)
- U2001 pad 22: Net-(U1-Pad22) -> unconnected-(U2001-PA6-Pad22)
- U2001 pad 23: Net-(U1-Pad23) -> unconnected-(U2001-PA7-Pad23)
- U2001 pad 24: Net-(U1-Pad24) -> unconnected-(U2001-PC4-Pad24)
- U2001 pad 25: Net-(U1-Pad25) -> unconnected-(U2001-PC5-Pad25)
- U2001 pad 26: Net-(U1-Pad26) -> unconnected-(U2001-PB0-Pad26)
- U2001 pad 27: Net-(U1-Pad27) -> unconnected-(U2001-PB1-Pad27)
- U2001 pad 29: Net-(U1-Pad29) -> unconnected-(U2001-PB10-Pad29)
- U2001 pad 33: Net-(U1-Pad33) -> unconnected-(U2001-PB12-Pad33)
- U2001 pad 34: Net-(U1-Pad34) -> unconnected-(U2001-PB13-Pad34)
- U2001 pad 35: Net-(U1-Pad35) -> unconnected-(U2001-PB14-Pad35)
- U2001 pad 36: Net-(U1-Pad36) -> unconnected-(U2001-PB15-Pad36)
- U2001 pad 37: Net-(U1-Pad37) -> unconnected-(U2001-PC6-Pad37)
- U2001 pad 38: Net-(U1-Pad38) -> unconnected-(U2001-PC7-Pad38)
- U2001 pad 39: Net-(U1-Pad39) -> unconnected-(U2001-PC8-Pad39)
- U2001 pad 4: Net-(U1-Pad4) -> unconnected-(U2001-PC15-Pad4)
- U2001 pad 40: Net-(U1-Pad40) -> unconnected-(U2001-PC9-Pad40)
- U2001 pad 44: Net-(U1-Pad44) -> unconnected-(U2001-PA11-Pad44)
- U2001 pad 45: Net-(U1-Pad45) -> unconnected-(U2001-PA12-Pad45)
- U2001 pad 49: Net-(U1-Pad49) -> unconnected-(U2001-PA14-Pad49)
- U2001 pad 5: Net-(U1-Pad5) -> unconnected-(U2001-PH0-Pad5)
- U2001 pad 50: Net-(U1-Pad50) -> unconnected-(U2001-PA15-Pad50)
- U2001 pad 51: Net-(U1-Pad51) -> unconnected-(U2001-PC10-Pad51)
- U2001 pad 52: Net-(U1-Pad52) -> unconnected-(U2001-PC11-Pad52)
- U2001 pad 53: Net-(U1-Pad53) -> unconnected-(U2001-PC12-Pad53)
- U2001 pad 54: Net-(U1-Pad54) -> unconnected-(U2001-PD2-Pad54)
- U2001 pad 55: Net-(U1-Pad55) -> unconnected-(U2001-PB3-Pad55)
- U2001 pad 56: Net-(U1-Pad56) -> unconnected-(U2001-PB4-Pad56)
- U2001 pad 57: Net-(U1-Pad57) -> unconnected-(U2001-PB5-Pad57)
- U2001 pad 58: Net-(U1-Pad58) -> unconnected-(U2001-PB6-Pad58)
- U2001 pad 59: Net-(U1-Pad59) -> unconnected-(U2001-PB7-Pad59)
- U2001 pad 6: Net-(U1-Pad6) -> unconnected-(U2001-PH1-Pad6)
- U2001 pad 61: Net-(U1-Pad61) -> unconnected-(U2001-PB8-Pad61)
- U2001 pad 62: Net-(U1-Pad62) -> unconnected-(U2001-PB9-Pad62)
- U2001 pad 8: Net-(U1-Pad8) -> unconnected-(U2001-PC0-Pad8)
- U2001 pad 9: Net-(U1-Pad9) -> unconnected-(U2001-PC1-Pad9)
- U6001 pad 10: Net-(U2-Pad10) -> unconnected-(U6001-DCD-Pad10)
- U6001 pad 11: Net-(U2-Pad11) -> unconnected-(U6001-CTS-Pad11)
- U6001 pad 12: Net-(U2-Pad12) -> unconnected-(U6001-CBUS4-Pad12)
- U6001 pad 13: Net-(U2-Pad13) -> unconnected-(U6001-CBUS2-Pad13)
- U6001 pad 14: Net-(U2-Pad14) -> unconnected-(U6001-CBUS3-Pad14)
- U6001 pad 19: Net-(U2-Pad19) -> unconnected-(U6001-~{RESET}-Pad19)
- U6001 pad 2: Net-(U2-Pad2) -> unconnected-(U6001-DTR-Pad2)
- U6001 pad 22: Net-(U2-Pad22) -> unconnected-(U6001-CBUS1-Pad22)
- U6001 pad 23: Net-(U2-Pad23) -> unconnected-(U6001-CBUS0-Pad23)
- U6001 pad 27: Net-(U2-Pad27) -> unconnected-(U6001-OSCI-Pad27)
- U6001 pad 28: Net-(U2-Pad28) -> unconnected-(U6001-OSCO-Pad28)
- U6001 pad 3: Net-(U2-Pad3) -> unconnected-(U6001-RTS-Pad3)
- U6001 pad 6: Net-(U2-Pad6) -> unconnected-(U6001-RI-Pad6)
- U6001 pad 9: Net-(U2-Pad9) -> unconnected-(U6001-DCR-Pad9)
